File: circuit/circuit.kicad_pcb (KiCad board)
At the start: 2 copper layers, 71.7 x 20 mm, 33 parts, among them J1 USB_A, U1 RP2040, U2 AMS1117-3.3, U3 W25Q32JVSS, U4 W25Q32JVSS, Y1 12MHz

Commit message: PCB v2
Parts:
- C1, R3, U2: moved to B.Cu
- moved SW1 43.6 mm to (146.6, 103.7), turned to 0 degrees
- moved R5 20.7 mm to (143.6, 103.9), turned to -90 degrees
- moved D1 20.5 mm to (143.6, 108.0), turned to 90 degrees
- moved C10 4.80 mm to (116.0, 107.9)
- moved C11 4.80 mm to (114.0, 107.9)
- moved C12 4.80 mm to (112.0, 107.9)
- moved C14 4.80 mm to (110.0, 107.9)
- moved C2 4.80 mm to (126.0, 107.9)
- moved C6 4.80 mm to (124.0, 107.9)
- moved C7 4.80 mm to (122.0, 107.9)
- moved C8 4.80 mm to (120.0, 107.9)
- moved C9 4.80 mm to (118.0, 107.9)
- moved R8 4.46 mm to (117.5, 103.3), turned to 0 degrees
- moved U2 4.37 mm to (152.2, 95.0), turned to -90 degrees
- moved C13 3.87 mm to (139.2, 103.7)
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Other:
- board size 71.7 x 20 mm -> 55.1 x 20 mm

Commit message: PCB v2
Parts:
- moved C16 10.8 mm to (131.0, 95.3)
- moved C15 10.8 mm to (134.2, 91.5)
- moved J2 10.8 mm to (122.1, 98.5)
- moved R4 10.8 mm to (134.2, 94.5)
- moved R7 10.8 mm to (123.8, 101.2)
- moved C1 10.8 mm to (167.6, 91.3)
- moved C10 10.8 mm to (126.6, 105.8)
- moved C11 10.8 mm to (124.6, 105.8)
- moved C12 10.8 mm to (122.6, 105.8)
- moved C14 10.8 mm to (120.6, 105.8)
- moved C2 10.8 mm to (136.6, 105.8)
- moved C6 10.8 mm to (134.6, 105.8)
- moved C7 10.8 mm to (132.6, 105.8)
- moved C8 10.8 mm to (130.6, 105.8)
- moved C9 10.8 mm to (128.6, 105.8)
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
Commit message: finalize PCB
Parts:
- C1, R3, U2, U3, U4: moved to F.Cu
- moved C2 16.2 mm to (120.4, 106.6), turned to 90 degrees
- moved C14 15.8 mm to (136.4, 106.6), turned to 90 degrees
- moved C6 12.2 mm to (122.4, 106.6), turned to 90 degrees
- moved C12 11.8 mm to (134.4, 106.6), turned to 90 degrees
- moved C16 10.2 mm to (121.1, 93.0), turned to 0 degrees
- moved R4 9.55 mm to (124.8, 93.0)
- moved Y1 9.54 mm to (121.0, 89.6)
- moved C15 9.47 mm to (124.8, 90.7)
- moved C7 8.24 mm to (124.4, 106.6), turned to 90 degrees
- moved R3 8.01 mm to (144.2, 88.8), turned to 180 degrees
- moved C11 7.84 mm to (132.4, 106.6), turned to 90 degrees
- moved R8 6.20 mm to (126.6, 95.2)
- moved R5 5.04 mm to (154.2, 106.8), turned to 90 degrees
- moved C13 4.70 mm to (145.2, 100.4), turned to 180 degrees
- moved C8 4.28 mm to (126.4, 106.6), turned to 90 degrees
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Routing:
- net +3V3: track 0.00 -> 160.6 mm, vias 0 -> 4
- net /DBG_BOOT: track 0.00 -> 54.7 mm, vias 0 -> 2
- net /IO_LED: track 0.00 -> 52.0 mm, vias 0 -> 2
- net /IO_BTN: track 0.00 -> 43.0 mm, vias 0 -> 1
- net /DBG_LED: track 0.00 -> 36.5 mm
- net /XIN: track 0.00 -> 22.9 mm
- net +1V1: track 0.00 -> 22.4 mm
- net Net-(J1-D-): track 0.00 -> 20.6 mm
- net Net-(J1-D+): track 0.00 -> 20.2 mm
- net /PMEM_IO1: track 0.00 -> 15.7 mm
- net /DMEM_CS: track 0.00 -> 15.2 mm
- net /PMEM_IO3: track 0.00 -> 14.3 mm
- net /DMEM_DO: track 0.00 -> 14.2 mm
- net VBUS: track 0.00 -> 14.1 mm
- net /XOUT: track 0.00 -> 13.8 mm
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Other:
- board size 55.1 x 20 mm -> 55.5 x 22 mm

Commit message: Final PCB fixes
Parts:
- moved C15 0.50 mm to (124.8, 90.2), turned to -90 degrees
- moved C16 0.50 mm to (121.0, 93.5)
- moved Y1 0.50 mm to (121.0, 90.1)
- moved R4 0.11 mm to (124.7, 93.0)
Routing:
- net /XIN: track 22.9 -> 23.9 mm
- net /PMEM_IO2: track 13.7 -> 14.5 mm
- net GND: vias 1 -> 2
